File: kicad/PwrBank/PwrBank.sch (KiCad schematic (older format))
At the start: 6 parts, among them J1 SCREW_TERMINALS_DCDC_MODULE, J2 CHARGEPORT, J3 BMS_UART, J4 SAFE_SHUTDOWN_WARNING, J5 OLED_CONN

Commit message: Work on schematic+implement capacitive feature using TOUCH0
Parts:
- removed J4: SAFE_SHUTDOWN_WARNING, Connector_JST:JST_XH_B2B-XH-A_1x02_P2.50mm_Vertical, symbol Connector:Conn_01x02_Female
- added J3: UART_COMMS_CON, Connector_JST:JST_XH_B4B-XH-A_1x04_P2.50mm_Vertical, symbol Connector:Conn_01x04_Female
- J1: footprint (none) -> TB003-500-P04BE:CUI_TB003-500-P04BE
- renumbered J3 to J4
Connections:
- net ESP32_AND_SUCH/SAFE_SHUTDOWN_SIGNAL: now also J3.2 (Pin_2)
- net GND: now also J3.1 (Pin_1)
- net +12V renamed +VDC
- new net ESP32_AND_SUCH/U1RXD: J3.3 (Pin_3)
- new net ESP32_AND_SUCH/U1TXD: J3.4 (Pin_4)
Other:
- note added: "Used for charging powerbank \nfrom VDC source"
- note removed: "Used for charging powerbank \nfrom 12V source."
Changed lines of the file:
@@
 Comment4 ""
 $EndDescr
-$Sheet
-S 600  700  650  600
-U 60EAFEE2
-F0 "MomentaryRGBSwitch" 50
-F1 "MomentaryRGBSwitch.sch" 50
-F2 "LED_R" I R 1250 800 50
-F3 "LED_G" I R 1250 900 50
-F4 "LED_B" I R 1250 1000 50
-F5 "BUTTON_NC" O R 1250 1100 50
-F6 "BUTTON_NO" O R 1250 1200 50
-$EndSheet
-NoConn ~ 1250 1100
-Text GLabel 1250 1200 2    50   Input ~ 0
+NoConn ~ 1450 1100
+Text GLabel 1450 1200 2    50   Input ~ 0
 BTN_NO
 $Sheet
@@
 	1250 2800 1300 2800
 $Sheet
-S 3400 1050 900  750
+S 3200 1150 900  750
 U 60EE26E7
 F0 "SmartSoftLatch" 50
 F1 "SmartSoftLatch.sch" 50
-F2 "BTN_NO" I R 4300 1500 50
-F3 "MCU_LATCH_BTN" O R 4300 1600 50
-F4 "MCU_LATCH_ENABLE" I R 4300 1700 50
-$EndSheet
-Text GLabel 4450 1500 2    50   Output ~ 0
+F2 "BTN_NO" I R 4100 1600 50
+F3 "MCU_LATCH_BTN" O R 4100 1700 50
+F4 "MCU_LATCH_ENABLE" I R 4100 1800 50
+$EndSheet
+Text GLabel 4250 1600 2    50   Output ~ 0
 BTN_NO
 Wire Wire Line
-	4450 1500 4300 1500
+	4250 1600 4100 1600
 Wire Wire Line
 	1300 2700 1250 2700
@@
 $EndSheet
 Text Notes 3250 4300 0    50   ~ 0
-Used for charging powerbank \nfrom 12V source.
+Used for charging powerbank \nfrom VDC source
 $Sheet
 S 3200 2200 2200 1050
@@
 F2 "BMS_TX" O R 5400 2400 50
 F3 "BMS_RX" I R 5400 2300 50
-F4 "SAFE_SHUTDOWN_SIGNAL" O R 5400 2650 50
+F4 "SAFE_SHUTDOWN_SIGNAL" O L 3200 3150 50
 F5 "SOFTLATCH_GATE_ENABLE" O L 3200 2600 50
 F6 "SDA1" B R 5400 3050 50
@@
 F9 "SCL2" O R 5400 2850 50
 F10 "SDA2" B R 5400 2750 50
+F11 "U1TXD" O L 3200 2950 50
+F12 "U1RXD" I L 3200 3050 50
+F13 "TOUCH_SENSE" O L 3200 2400 50
 $EndSheet
 Text GLabel 3100 2600 0    50   Input ~ 0
@@
 Wire Wire Line
 	3100 2600 3200 2600
-Text GLabel 4450 1700 2    50   Output ~ 0
+Text GLabel 4250 1800 2    50   Output ~ 0
 MCU_LATCH_EN
 Wire Wire Line
-	4450 1700 4300 1700
+	4250 1800 4100 1800
 Text GLabel 3100 2750 0    50   Output ~ 0
 MCU_LATCH_BTN
@@
 	3100 2750 3200 2750
 Wire Wire Line
-	4450 1600 4300 1600
-Text GLabel 4450 1600 2    50   Input ~ 0
+	4250 1700 4100 1700
+Text GLabel 4250 1700 2    50   Input ~ 0
 MCU_LATCH_BTN
-Wire Wire Line
-	5400 2650 5950 2650
-Wire Wire Line
-	5950 2650 5950 2600
-Wire Wire Line
-	5950 2600 6050 2600
-$Comp
-L Connector:Conn_01x04_Female J3
+$Comp
+L Connector:Conn_01x04_Female J4
 U 1 1 60F67167
 P 5800 1400
-F 0 "J3" V 5738 1112 50  0000 R CNN
+F 0 "J4" V 5738 1112 50  0000 R CNN
 F 1 "BMS_UART" V 5647 1112 50  0000 R CNN
 F 2 "Connector_JST:JST_XH_B4B-XH-A_1x04_P2.50mm_Vertical" H 5800 1400 50  0001 C CNN
@@
 Text Notes 600  3400 0    50   ~ 10
 BMS Battery in port and charging port.
-Text GLabel 1300 800  2    50   Output ~ 0
+Text GLabel 1500 800  2    50   Output ~ 0
 LEDRING_R
 Wire Wire Line
-	1300 800  1250 800
+	1500 800  1450 800
 $Comp
 L power:+BATT #PWR03
@@
 $EndComp
 $Comp
-L power:+12V #PWR02
-U 1 1 60FEFA09
-P 1150 4250
-F 0 "#PWR02" H 1150 4100 50  0001 C CNN
-F 1 "+12V" V 1165 4378 50  0000 L CNN
-F 2 "" H 1150 4250 50  0001 C CNN
-F 3 "" H 1150 4250 50  0001 C CNN
-	1    1150 4250
-	0    -1   -1   0
-$EndComp
-$Comp
 L power:GND #PWR01
 U 1 1 60FF3549
@@
 F 0 "J1" H 942 1775 50  0000 C CNN
 F 1 "SCREW_TERMINALS_DCDC_MODULE" H 942 1866 50  0000 C CNN
-F 2 "" H 1050 2200 50  0001 C CNN
-F 3 "~" H 1050 2200 50  0001 C CNN
+F 2 "TB003-500-P04BE:CUI_TB003-500-P04BE" H 1050 2200 50  0001 C CNN
+F 3 "https://nl.mouser.com/datasheet/2/670/tb003_500-2306959.pdf" H 1050 2200 50  0001 C CNN
 	1    1050 2200
 	-1   0    0    1
@@
 P 5700 1750
 AR Path="/60ECA2F7/610A7150" Ref="#PWR?"  Part="1"
-AR Path="/610A7150" Ref="#PWR010"  Part="1"
-F 0 "#PWR010" H 5700 1500 50  0001 C CNN
+AR Path="/610A7150" Ref="#PWR011"  Part="1"
+F 0 "#PWR011" H 5700 1500 50  0001 C CNN
 F 1 "GND" H 5705 1577 50  0000 C CNN
 F 2 "" H 5700 1750 50  0001 C CNN
@@
 $EndComp
 $Comp
-L Connector:Conn_01x02_Female J4
-U 1 1 60F64EEF
-P 6250 2500
-F 0 "J4" H 6278 2476 50  0000 L CNN
-F 1 "SAFE_SHUTDOWN_WARNING" H 6278 2385 50  0000 L CNN
-F 2 "Connector_JST:JST_XH_B2B-XH-A_1x02_P2.50mm_Vertical" H 6250 2500 50  0001 C CNN
-F 3 "~" H 6250 2500 50  0001 C CNN
-	1    6250 2500
-	1    0    0    -1
-$EndComp
-$Comp
 L power:GND #PWR?
 U 1 1 610A84AF
 P 6050 2500
 AR Path="/60ECA2F7/610A84AF" Ref="#PWR?"  Part="1"
-AR Path="/610A84AF" Ref="#PWR011"  Part="1"
-F 0 "#PWR011" H 6050 2250 50  0001 C CNN
+AR Path="/610A84AF" Ref="#PWR012"  Part="1"
+F 0 "#PWR012" H 6050 2250 50  0001 C CNN
 F 1 "GND" V 6055 2372 50  0000 R CNN
 F 2 "" H 6050 2500 50  0001 C CNN
@@
 	5400 2850 6150 2850
 $Comp
-L power:+3.3V #PWR012
+L power:+3.3V #PWR013
 U 1 1 60FA2045
 P 6150 2950
-F 0 "#PWR012" H 6150 2800 50  0001 C CNN
+F 0 "#PWR013" H 6150 2800 50  0001 C CNN
 F 1 "+3.3V" V 6165 3078 50  0000 L CNN
 F 2 "" H 6150 2950 50  0001 C CNN
@@
 $EndComp
 $Comp
-L power:GND #PWR013
+L power:GND #PWR014
 U 1 1 60FA2D4B
 P 6150 3050
-F 0 "#PWR013" H 6150 2800 50  0001 C CNN
+F 0 "#PWR014" H 6150 2800 50  0001 C CNN
 F 1 "GND" V 6155 2922 50  0000 R CNN
 F 2 "" H 6150 3050 50  0001 C CNN
@@
 Wire Wire Line
 	6200 3900 6250 3900
-Text GLabel 1300 900  2    50   Output ~ 0
+Text GLabel 1500 900  2    50   Output ~ 0
 LEDRING_G
-Text GLabel 1300 1000 2    50   Output ~ 0
+Text GLabel 1500 1000 2    50   Output ~ 0
 LEDRING_B
 Wire Wire Line
-	1250 900  1300 900
-Wire Wire Line
-	1250 1000 1300 1000
+	1450 900  1500 900
+Wire Wire Line
+	1450 1000 1500 1000
+$Comp
+L power:+VDC #PWR02
+U 1 1 60FDC35F
+P 1150 4250
+F 0 "#PWR02" H 1150 4150 50  0001 C CNN
+F 1 "+VDC" V 1150 4479 50  0000 L CNN
+F 2 "" H 1150 4250 50  0001 C CNN
+F 3 "" H 1150 4250 50  0001 C CNN
+	1    1150 4250
+	0    -1   -1   0
+$EndComp
+$Comp
+L Connector:Conn_01x04_Female J3
+U 1 1 60FE873B
+P 2600 3150
+F 0 "J3" H 2800 3050 50  0000 C CNN
+F 1 "UART_COMMS_CON" H 2950 3150 50  0000 C CNN
+F 2 "Connector_JST:JST_XH_B4B-XH-A_1x04_P2.50mm_Vertical" H 2600 3150 50  0001 C CNN
+F 3 "~" H 2600 3150 50  0001 C CNN
+	1    2600 3150
+	-1   0    0    1
+$EndComp
+Wire Wire Line
+	2800 2950 3200 2950
+Wire Wire Line
+	2800 3050 3200 3050
+Wire Wire Line
+	2800 3150 3200 3150
+$Comp
+L power:GND #PWR010
+U 1 1 60FED4F1
+P 2900 3250
+F 0 "#PWR010" H 2900 3000 50  0001 C CNN
+F 1 "GND" V 2905 3122 50  0000 R CNN
+F 2 "" H 2900 3250 50  0001 C CNN
+F 3 "" H 2900 3250 50  0001 C CNN
+	1    2900 3250
+	0    -1   -1   0
+$EndComp
+Wire Wire Line
+	2900 3250 2800 3250
+$Sheet
+S 600  700  850  700
+U 60EAFEE2
+F0 "MomentaryRGBSwitch" 50
+F1 "MomentaryRGBSwitch.sch" 50
+F2 "LED_R" I R 1450 800 50
+F3 "LED_G" I R 1450 900 50
+F4 "LED_B" I R 1450 1000 50
+F5 "BUTTON_NC" O R 1450 1100 50
+F6 "BUTTON_NO" O R 1450 1200 50
+F7 "CAPACITIVE_SENSE" O R 1450 1300 50
+$EndSheet
+Text GLabel 1500 1300 2    50   Output ~ 0
+CAPACITIVE_BTN_SENSE
+Wire Wire Line
+	1500 1300 1450 1300
+Text GLabel 3150 2400 0    50   Input ~ 0
+CAPACITIVE_BTN_SENSE
+Wire Wire Line
+	3200 2400 3150 2400
 $EndSCHEMATC
